File: BS/schematic/2rfm69.sch (EAGLE design)
At the start: 17 parts, among them IC1 Atmega328P-PU, IC2 FT232R, Q1 16MHz, U1 RFM69, X1 PN61729-S

Commit message: Test schematic BS
Parts:
- added C6: 10uF, rcl:CPOL-EUE2,5-6E
- added F1: 500mA, fuse:TE5
- added U$1: LM1117, 1117:LM1117
Connections:
- new net 3V3_FTDI: IC2.3V3OUT, IC2.VCCIO
- new net N$5: LED1.C, R3.2
- new net N$8: F1.2, X1.1
- net +3V3: now also C6.+, LED1.A, SV2.2, U$1.OUT
- net +5V: now also F1.1, SV2.1, U$1.IN; no longer X1.1
- net D6: now also SV2.5
- net D7: now also SV2.6
- net GND: now also C6.-, R3.1, SV2.3, U$1.GND, U$1.GND1
Other:
- moved on the sheet: LED1, R3
Changed lines of the file:
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@@
 <part name="R3" library="rcl" deviceset="R-EU_" device="0204/7" value="1k"/>
 <part name="LED1" library="led" deviceset="LED" device="3MM"/>
+<part name="U$1" library="1117" deviceset="LM1117" device=""/>
+<part name="GND7" library="supply1" deviceset="GND" device=""/>
+<part name="C6" library="rcl" deviceset="CPOL-EU" device="E2,5-6E" value="10uF"/>
+<part name="F1" library="fuse" deviceset="TE5" device="" value="500mA"/>
 </parts>
 <sheets>
@@
 <attribute name="VALUE" x="111.379" y="9.144" size="1.778" layer="96" rot="R180"/>
 </instance>
-<instance part="R3" gate="G$1" x="157.48" y="0" smashed="yes" rot="R90">
-<attribute name="NAME" x="155.9814" y="-3.81" size="1.778" layer="95" rot="R90"/>
-<attribute name="VALUE" x="160.782" y="-3.81" size="1.778" layer="96" rot="R90"/>
-</instance>
-<instance part="LED1" gate="G$1" x="144.78" y="0"/>
+<instance part="R3" gate="G$1" x="185.42" y="-17.78" smashed="yes" rot="R90">
+<attribute name="NAME" x="183.9214" y="-21.59" size="1.778" layer="95" rot="R90"/>
+<attribute name="VALUE" x="188.722" y="-21.59" size="1.778" layer="96" rot="R90"/>
+</instance>
+<instance part="LED1" gate="G$1" x="185.42" y="-5.08"/>
+<instance part="U$1" gate="G$1" x="154.94" y="-5.08"/>
+<instance part="GND7" gate="1" x="134.62" y="-27.94"/>
+<instance part="C6" gate="G$1" x="175.26" y="-10.16"/>
+<instance part="F1" gate="1" x="12.7" y="-20.32" rot="R90"/>
 </instances>
 <busses>
@@
 <wire x1="91.44" y1="88.9" x2="91.44" y2="91.44" width="0.1524" layer="91"/>
 </segment>
+<segment>
+<pinref part="U$1" gate="G$1" pin="OUT"/>
+<label x="170.18" y="-2.54" size="1.778" layer="95"/>
+<wire x1="170.18" y1="-2.54" x2="175.26" y2="-2.54" width="0.1524" layer="91"/>
+<pinref part="C6" gate="G$1" pin="+"/>
+<wire x1="175.26" y1="-2.54" x2="175.26" y2="-7.62" width="0.1524" layer="91"/>
+<pinref part="LED1" gate="G$1" pin="A"/>
+<wire x1="175.26" y1="-2.54" x2="185.42" y2="-2.54" width="0.1524" layer="91"/>
+<junction x="175.26" y="-2.54"/>
+</segment>
+<segment>
+<pinref part="SV2" gate="1" pin="2"/>
+<wire x1="-20.32" y1="-7.62" x2="-15.24" y2="-7.62" width="0.1524" layer="91"/>
+<label x="-20.32" y="-7.62" size="1.778" layer="95"/>
+</segment>
 </net>
 <net name="GND" class="0">
@@
 <pinref part="C1" gate="G$1" pin="1"/>
 <junction x="-40.64" y="58.42"/>
-<pinref part="C2" gate="G$1" pin="1"/>
-<wire x1="-27.94" y1="60.96" x2="-30.48" y2="60.96" width="0.1524" layer="91"/>
 <wire x1="-30.48" y1="60.96" x2="-30.48" y2="55.88" width="0.1524" layer="91"/>
-<pinref part="C3" gate="G$1" pin="1"/>
 <wire x1="-30.48" y1="55.88" x2="-30.48" y2="48.26" width="0.1524" layer="91"/>
 <wire x1="-30.48" y1="48.26" x2="-30.48" y2="35.56" width="0.1524" layer="91"/>
-<wire x1="-27.94" y1="55.88" x2="-30.48" y2="55.88" width="0.1524" layer="91"/>
-<junction x="-30.48" y="55.88"/>
 <pinref part="IC1" gate="G$1" pin="GND@1"/>
 <wire x1="-12.7" y1="48.26" x2="-30.48" y2="48.26" width="0.1524" layer="91"/>
 <junction x="-30.48" y="48.26"/>
+<pinref part="C3" gate="G$1" pin="1"/>
+<wire x1="-27.94" y1="55.88" x2="-30.48" y2="55.88" width="0.1524" layer="91"/>
+<junction x="-30.48" y="55.88"/>
+<pinref part="C2" gate="G$1" pin="1"/>
+<wire x1="-27.94" y1="60.96" x2="-30.48" y2="60.96" width="0.1524" layer="91"/>
 </segment>
 <segment>
@@
 <pinref part="GND6" gate="1" pin="GND"/>
 </segment>
+<segment>
+<wire x1="134.62" y1="-22.86" x2="149.86" y2="-22.86" width="0.1524" layer="91"/>
+<pinref part="GND7" gate="1" pin="GND"/>
+<wire x1="149.86" y1="-22.86" x2="160.02" y2="-22.86" width="0.1524" layer="91"/>
+<wire x1="160.02" y1="-22.86" x2="175.26" y2="-22.86" width="0.1524" layer="91"/>
+<wire x1="134.62" y1="-22.86" x2="134.62" y2="-25.4" width="0.1524" layer="91"/>
+<pinref part="U$1" gate="G$1" pin="GND"/>
+<wire x1="149.86" y1="-17.78" x2="149.86" y2="-22.86" width="0.1524" layer="91"/>
+<junction x="149.86" y="-22.86"/>
+<pinref part="U$1" gate="G$1" pin="GND1"/>
+<wire x1="160.02" y1="-17.78" x2="160.02" y2="-22.86" width="0.1524" layer="91"/>
+<junction x="160.02" y="-22.86"/>
+<pinref part="C6" gate="G$1" pin="-"/>
+<wire x1="175.26" y1="-22.86" x2="175.26" y2="-15.24" width="0.1524" layer="91"/>
+<wire x1="175.26" y1="-22.86" x2="185.42" y2="-22.86" width="0.1524" layer="91"/>
+<junction x="175.26" y="-22.86"/>
+<pinref part="R3" gate="G$1" pin="1"/>
+</segment>
+<segment>
+<pinref part="SV2" gate="1" pin="3"/>
+<wire x1="-20.32" y1="-5.08" x2="-15.24" y2="-5.08" width="0.1524" layer="91"/>
+<label x="-20.32" y="-5.08" size="1.778" layer="95"/>
+</segment>
 </net>
 <net name="N$1" class="0">
@@
 <label x="35.56" y="38.1" size="1.778" layer="95"/>
 </segment>
+<segment>
+<pinref part="SV2" gate="1" pin="6"/>
+<wire x1="-20.32" y1="2.54" x2="-15.24" y2="2.54" width="0.1524" layer="91"/>
+<label x="-20.32" y="2.54" size="1.778" layer="95"/>
+</segment>
 </net>
 <net name="D6" class="0">
@@
 <label x="35.56" y="40.64" size="1.778" layer="95"/>
 </segment>
+<segment>
+<pinref part="SV2" gate="1" pin="5"/>
+<wire x1="-20.32" y1="0" x2="-15.24" y2="0" width="0.1524" layer="91"/>
+<label x="-20.32" y="0" size="1.778" layer="95"/>
+</segment>
 </net>
 <net name="D5" class="0">
@@
 <net name="+5V" class="0">
 <segment>
-<pinref part="X1" gate="G$1" pin="1"/>
-<wire x1="12.7" y1="-7.62" x2="12.7" y2="-12.7" width="0.1524" layer="91"/>
-<wire x1="2.54" y1="-12.7" x2="2.54" y2="2.54" width="0.1524" layer="91"/>
+<wire x1="2.54" y1="-30.48" x2="2.54" y2="2.54" width="0.1524" layer="91"/>
 <pinref part="VIN" gate="1" pin="+5V"/>
-<wire x1="2.54" y1="-12.7" x2="12.7" y2="-12.7" width="0.1524" layer="91"/>
-<wire x1="12.7" y1="-12.7" x2="12.7" y2="-30.48" width="0.1524" layer="91"/>
 <wire x1="12.7" y1="-30.48" x2="58.42" y2="-30.48" width="0.1524" layer="91"/>
 <wire x1="58.42" y1="-30.48" x2="58.42" y2="22.86" width="0.1524" layer="91"/>
 <pinref part="IC2" gate="1" pin="VCC"/>
 <wire x1="58.42" y1="22.86" x2="71.12" y2="22.86" width="0.1524" layer="91"/>
+<pinref part="F1" gate="1" pin="1"/>
+<wire x1="12.7" y1="-25.4" x2="12.7" y2="-30.48" width="0.1524" layer="91"/>
+<wire x1="2.54" y1="-30.48" x2="12.7" y2="-30.48" width="0.1524" layer="91"/>
+<junction x="12.7" y="-30.48"/>
+</segment>
+<segment>
+<pinref part="U$1" gate="G$1" pin="IN"/>
+<wire x1="139.7" y1="-2.54" x2="134.62" y2="-2.54" width="0.1524" layer="91"/>
+<label x="134.62" y="-2.54" size="1.778" layer="95"/>
+</segment>
+<segment>
+<pinref part="SV2" gate="1" pin="1"/>
+<wire x1="-20.32" y1="-10.16" x2="-15.24" y2="-10.16" width="0.1524" layer="91"/>
+<label x="-20.32" y="-10.16" size="1.778" layer="95"/>
 </segment>
 </net>
@@
 </segment>
 </net>
+<net name="N$5" class="0">
+<segment>
+<pinref part="LED1" gate="G$1" pin="C"/>
+<pinref part="R3" gate="G$1" pin="2"/>
+<wire x1="185.42" y1="-10.16" x2="185.42" y2="-12.7" width="0.1524" layer="91"/>
+</segment>
+</net>
+<net name="N$8" class="0">
+<segment>
+<pinref part="X1" gate="G$1" pin="1"/>
+<pinref part="F1" gate="1" pin="2"/>
+<wire x1="12.7" y1="-7.62" x2="12.7" y2="-15.24" width="0.1524" layer="91"/>
+</segment>
+</net>
+<net name="3V3_FTDI" class="0">
+<segment>
+<pinref part="IC2" gate="1" pin="VCCIO"/>
+<wire x1="71.12" y1="20.32" x2="66.04" y2="20.32" width="0.1524" layer="91"/>
+<label x="60.96" y="20.32" size="1.778" layer="95"/>
+</segment>
+<segment>
+<pinref part="IC2" gate="1" pin="3V3OUT"/>
+<wire x1="71.12" y1="-5.08" x2="66.04" y2="-5.08" width="0.1524" layer="91"/>
+<label x="58.42" y="-5.08" size="1.778" layer="95"/>
+</segment>
+</net>
