File: drone/schematic/schematic_test/bs_prod.brd (EAGLE design)
At the start: 95 x 50 mm, 29 parts, among them U1 ATMEGA328P_PDIP, U2 RFM69HW, U3 RFM69HW, Y1 16MHz

Commit message: production drone schematic
Parts:
- removed LED1, LED2, LED3: (no value), SparkFun-LED:LED-1206
- added 1_RX/TX, PWR_RF1, PWR_RF2, RF2_RX/TX: (no value), SparkFun-LED:LED-1206
- added C10, C11: 0.47uF, SparkFun-Capacitors:1206
- added JP1: (no value), SparkFun-Connectors:1X04
- added R6: 1k, SparkFun-Resistors:1206
- added SW1: 418117270902, Eagle_Wuerth_Elektronik_Switch:418117270902
- moved R4 40.1 mm to (15.5, 2.97), turned to 180 degrees
- moved R5 40.0 mm to (15.0, 47.0), turned to 180 degrees
- moved R3 8.00 mm to (38.0, 47.0)
- moved RESET 4.52 mm to (86.2, 41.3)
- renumbered SMA to SMA_RF1, SMA1 to SMA_RF2
Connections:
- new net D8: JP1.3, U1.14
- new net N$18: R3.2, U1.15
- new net N$19: C5.1, PWR_RF2.A, SW1.1, U3.8
- new net N$21: C9.1, PWR_RF1.A, SW1.2, U2.8
- net 3.3V: now also C10.1, C11.1, JP1.4, SW1.3, SW1.4; no longer C5.1, C9.1, LED1.A, LED3.A, U2.8, U3.8
- net A2: now also R6.2
- net D7: now also JP1.2
- net GND: now also 1_RX/TX.C, C10.2, C11.2, JP1.1, RF2_RX/TX.C; no longer LED2.C
- net N$12: now also 1_RX/TX.A
- net N$13: now also R6.1, RF2_RX/TX.A; no longer LED2.A, R3.2
- net N$20: now also PWR_RF1.C; no longer LED3.C
- net N$9: now also PWR_RF2.C; no longer LED1.C
Routing:
- net GND: track 376.1 -> 437.6 mm, vias 10 -> 13
- net N$19: track 0.00 -> 58.7 mm, vias 0 -> 1
- net N$21: track 0.00 -> 33.1 mm, vias 0 -> 1
- net N$18: track 0.00 -> 20.1 mm, vias 0 -> 1
- net A2: track 0.00 -> 19.0 mm
- net 3.3V: track 211.2 -> 193.5 mm, vias 2 -> 3
- net D7: track 0.00 -> 17.6 mm
- net D8: track 0.00 -> 13.7 mm
- net N$12: track 0.00 -> 7.10 mm
- net N$20: track 0.00 -> 6.08 mm
- net N$9: track 0.00 -> 4.98 mm
- net RST: track 49.2 -> 54.0 mm
- net N$13: track 0.00 -> 4.10 mm
- net N$8: track 37.6 -> 39.2 mm
- added copper zone on layer 1, net GND
- added copper zone on layer 16, net GND
Other:
- board text added: "D7"
- board text added: "D8"

Commit message: some fixed for drone schematic
Parts:
- moved C4 5.00 mm to (82.5, 29.0)
- moved C3 4.24 mm to (82.5, 26.2)
- moved Y1 3.16 mm to (75.4, 27.0)
- renumbered RF2_RX/TX to 2_RX/TX
Routing:
- net GND: track 437.6 -> 429.3 mm
- net N$6: track 15.6 -> 20.6 mm
- net N$7: track 16.4 -> 20.0 mm
- net 3.3V: track 193.5 -> 195.1 mm
- net D7: track 17.6 -> 18.4 mm
- net D13_SCK: track 40.9 -> 41.6 mm
- net D12_MISO: track 41.0 -> 41.6 mm
Other:
- board text added: "Matsepura A.M."
- board text added: "drone sch. rev.1.0"

Commit message: add main layout
Parts:
- C3, C4: value 20pF -> 22pF
- moved R5 7.81 mm to (20.0, 41.0)
- moved PWR_RF1 6.92 mm to (20.0, 46.9), turned to 180 degrees
- moved PWR_RF2 6.75 mm to (21.5, 5.05), turned to 0 degrees
- moved C4 5.20 mm to (82.5, 34.2)
- moved 1_RX/TX 3.00 mm to (31.0, 47.0)
- moved Y1 3.00 mm to (75.4, 30.0)
- moved R4 2.83 mm to (13.5, 4.97)
- moved C6 2.08 mm to (80.4, 18.5), turned to 270 degrees
- moved SMA_RF1 2.00 mm to (6.09, 35.7)
- moved C7 1.91 mm to (85.5, 18.4), turned to 270 degrees
- moved C8 1.00 mm to (71.6, 18.0)
- moved RESET 1.00 mm to (85.2, 41.3)
- moved C3 0.30 mm to (82.5, 25.9)
Routing:
- net N$21: track 33.1 -> 41.0 mm
- net N$19: track 58.7 -> 65.4 mm
- net N$12: track 7.10 -> 4.10 mm
- net N$11: track 18.2 -> 15.5 mm
- net N$6: track 20.6 -> 18.0 mm
- net GND: track 429.3 -> 427.3 mm, vias 13 -> 12
- net 5V: track 15.0 -> 16.6 mm
- net RST: track 54.0 -> 55.4 mm
- net 3.3V: track 195.1 -> 193.9 mm
- net D2: track 72.0 -> 71.2 mm
- net N$8: track 39.2 -> 38.4 mm
- net N$7: track 20.0 -> 19.3 mm
Other:
- board text added: "Holostov K.M."

Commit message: current drone schematic
Connections:
- net D3: no longer U3.2
Routing:
- net D3: track 46.5 -> 45.9 mm
Changed lines of the file:
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@@
 </signal>
 <signal name="D3">
-<contactref element="U3" pad="2"/>
 <contactref element="U1" pad="5"/>
 <wire x1="63.6514" y1="15.7208" x2="59.8396" y2="19.5326" width="0.4064" layer="16"/>
@@
 <wire x1="28.3464" y1="19.5072" x2="22.2758" y2="19.5072" width="0.4064" layer="1"/>
 <wire x1="22.2758" y1="19.5072" x2="22.2512" y2="19.4826" width="0.4064" layer="1"/>
-<wire x1="22.2512" y1="19.4826" x2="21.7262" y2="19.4826" width="0.4064" layer="1"/>
 </signal>
 <signal name="N$24">
