File: drone/schematic/schematic_test/bs_prod.sch (EAGLE design)
At the start: 29 parts, among them U1 ATMEGA328P_PDIP, U2 RFM69HW, U3 RFM69HW, Y1 16MHz

Commit message: production drone schematic
Parts:
- removed LED2: (no value), SparkFun-LED:LED1206
- added 1_RX/TX, RF2_RX/TX: (no value), SparkFun-LED:LED1206
- added C10, C11: 0.47uF, SparkFun-Capacitors:CAP1206
- added JP1: (no value), SparkFun-Connectors:M04PTH
- added R6: 1k, SparkFun-Resistors:RESISTOR1206
- added SW1: 418117270902, Eagle_Wuerth_Elektronik_Switch:418117270902
- renumbered LED1 to PWR_RF2, LED3 to PWR_RF1, SMA to SMA_RF1, SMA1 to SMA_RF2
Connections:
- new net D8: JP1.3, U1.PB0(ICP)
- new net N$18: R3.2, U1.PB1(OC1A)
- new net N$19: C5.1, PWR_RF2.A, SW1.1, U3.3.3V
- new net N$21: C9.1, PWR_RF1.A, SW1.2, U2.3.3V
- net 3.3V: now also C10.1, C11.1, JP1.4, SW1.3, SW1.4; no longer C5.1, C9.1, PWR_RF1.A, PWR_RF2.A, U2.3.3V, U3.3.3V
- net A2: now also R6.2
- net D7: now also JP1.2
- net GND: now also 1_RX/TX.C, C10.2, C11.2, JP1.1, RF2_RX/TX.C; no longer LED2.C
- net N$12: now also 1_RX/TX.A
- net N$13: now also R6.1, RF2_RX/TX.A; no longer LED2.A, R3.2
Other:
- moved on the sheet: PWR, R2, R3

Commit message: some fixed for drone schematic
Parts:
- renumbered RF2_RX/TX to 2_RX/TX
Changed lines of the file:
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@@
 <part name="GND16" library="SparkFun-Aesthetics" deviceset="GND" device=""/>
 <part name="R6" library="SparkFun-Resistors" deviceset="RESISTOR" device="1206" value="1k"/>
-<part name="RF2_RX/TX" library="SparkFun-LED" deviceset="LED" device="1206"/>
+<part name="2_RX/TX" library="SparkFun-LED" deviceset="LED" device="1206"/>
 <part name="GND17" library="SparkFun-Aesthetics" deviceset="GND" device=""/>
 <part name="SW1" library="Eagle_Wuerth_Elektronik_Switch" deviceset="418117270902" device=""/>
@@
 <instance part="GND16" gate="1" x="165.1" y="127"/>
 <instance part="R6" gate="G$1" x="81.28" y="167.64"/>
-<instance part="RF2_RX/TX" gate="G$1" x="71.12" y="165.1"/>
+<instance part="2_RX/TX" gate="G$1" x="71.12" y="165.1"/>
 <instance part="GND17" gate="1" x="71.12" y="154.94"/>
 <instance part="SW1" gate="G$1" x="190.5" y="109.22" smashed="yes">
@@
 </segment>
 <segment>
-<pinref part="RF2_RX/TX" gate="G$1" pin="C"/>
+<pinref part="2_RX/TX" gate="G$1" pin="C"/>
 <pinref part="GND17" gate="1" pin="GND"/>
 <wire x1="71.12" y1="160.02" x2="71.12" y2="157.48" width="0.1524" layer="91"/>
@@
 <net name="N$13" class="0">
 <segment>
-<pinref part="RF2_RX/TX" gate="G$1" pin="A"/>
+<pinref part="2_RX/TX" gate="G$1" pin="A"/>
 <pinref part="R6" gate="G$1" pin="1"/>
 <wire x1="71.12" y1="167.64" x2="76.2" y2="167.64" width="0.1524" layer="91"/>

Commit message: add main layout
Parts:
- C3, C4: value 20pF -> 22pF
Changed lines of the file:
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@@
 <setting verticaltext="up"/>
 </settings>
-<grid distance="0.1" unitdist="inch" unit="inch" style="lines" multiple="1" display="yes" altdistance="0.01" altunitdist="inch" altunit="inch"/>
+<grid distance="0.1" unitdist="inch" unit="inch" style="lines" multiple="1" display="no" altdistance="0.01" altunitdist="inch" altunit="inch"/>
 <layers>
 <layer number="1" name="Top" color="4" fill="1" visible="no" active="no"/>
@@
 <part name="SUPPLY1" library="SparkFun-Aesthetics" deviceset="3.3V" device=""/>
 <part name="SUPPLY2" library="SparkFun-Aesthetics" deviceset="5V" device=""/>
-<part name="C3" library="SparkFun-Capacitors" deviceset="CAP" device="1206" value="20pF"/>
-<part name="C4" library="SparkFun-Capacitors" deviceset="CAP" device="1206" value="20pF"/>
+<part name="C3" library="SparkFun-Capacitors" deviceset="CAP" device="1206" value="22pF"/>
+<part name="C4" library="SparkFun-Capacitors" deviceset="CAP" device="1206" value="22pF"/>
 <part name="GND2" library="SparkFun-Aesthetics" deviceset="GND" device=""/>
 <part name="GND3" library="SparkFun-Aesthetics" deviceset="GND" device=""/>

Commit message: current drone schematic
Connections:
- new net N$2: U2.DIO0
- net D2: no longer U2.DIO0
- net D3: no longer U3.DIO0
Other:
- moved on the sheet: 1_RX/TX, 2_RX/TX, C1, C10, C3, C4, C5, C6, C8, C9, JP1, JP5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
